File: circuit/untitled.kicad_sch (KiCad schematic)
At the start: 28 parts, among them J1 RPi Zero female, J2 ISCP, J3 Conn_01x08, SW1 SW_SPDT, U1 ULN2803A, U2 74HC04

Commit message: .
Parts:
- added unit 7 of U2
- added U3: TXB0104D, Package_SO:SOIC-14_3.9x8.7mm_P1.27mm, symbol Logic_LevelTranslator:TXB0104D
Connections:
- net +3V3: now also U3.1 (VCCA)
- net +5V: now also R10.1, R11.1, R12.1, R13.1, R8.1, R9.1, U2.14 (VCC)
- net GND: now also U2.7 (GND), U3.7 (GND)
- net MISO: no longer J1.21 (Pin_21), J2.5 (Pin_5), R12.2, U2.11
- net TX: no longer J3.1 (Pin_1)
- net VCC: now also U3.14 (VCCB)
- net RX renamed RX_5V
- net RX_5V: now also U3.13 (B1); no longer J1.10 (Pin_10)
- new net MISO_3V3: J1.21 (Pin_21), U3.3 (A2)
- new net MISO_5V: J2.5 (Pin_5), R12.2, U2.11, U3.12 (B2)
- new net RX_3V3: J1.10 (Pin_10), U3.2 (A1)
- new net TX_5V: J3.1 (Pin_1)
- no-connect marks 5 -> 9
Other:
- note added: "<-"
- note added: "NOTCH"
